Commit message: added bug2

File: simulation_ws/src/i214_description/urdf/i214.xacro (robot description, xacro)
@@ -25,4 +25,17 @@
       <material name="blue"/>
     </visual>
+    <!-- camera mount -->
+    <collision name="collision_camera_mount">
+      <geometry>
+        <box size="0.1 0.3 0.1"/>
+      </geometry>
+    </collision>
+    <visual>
+      <origin rpy="0 0 0" xyz="0 0 0.05"/>
+      <geometry>
+        <box size="0.1 0.3 0.1"/>
+      </geometry>
+      <material name="blue"/>
+    </visual>
     <!-- caster front -->
     <collision name="caster_front_collision">
@@ -48,4 +61,31 @@
       </geometry>
     </visual>
+  </link>
+  <joint name="camera_joint" type="fixed">
+    <axis xyz="0 1 0" />
+    <origin xyz="0 0 0.15" rpy="0 0 0"/>
+    <parent link="link_chassis"/>
+    <child link="camera_link"/>
+  </joint>
+  <!-- Camera -->
+  <link name="camera_link">
+    <collision>
+      <origin xyz="0 0 0" rpy="0 0 0"/>
+      <geometry>
+        <box size="0.1 0.1 0.1"/>
+      </geometry>
+    </collision>
+    <visual>
+      <origin xyz="0 0 0" rpy="0 0 0"/>
+      <geometry>
+        <box size="0.1 0.1 0.1"/>
+      </geometry>
+      <material name="red"/>
+    </visual>
+    <inertial>
+      <mass value="1e-5" />
+      <origin xyz="0 0 0" rpy="0 0 0"/>
+      <inertia ixx="1e-6" ixy="0" ixz="0" iyy="1e-6" iyz="0" izz="1e-6" />
+    </inertial>
   </link>
   <link name="sensor_laser">

Commit message: dwa added

File: simulation_ws/src/i214_description/urdf/i214.xacro (robot description, xacro)
@@ -28,5 +28,5 @@
     <collision name="collision_camera_mount">
       <geometry>
-        <box size="0.1 0.3 0.1"/>
+        <box size="0.1 0.25 0.1"/>
       </geometry>
     </collision>
@@ -34,5 +34,5 @@
       <origin rpy="0 0 0" xyz="0 0 0.05"/>
       <geometry>
-        <box size="0.1 0.3 0.1"/>
+        <box size="0.1 0.25 0.1"/>
       </geometry>
       <material name="blue"/>
@@ -92,6 +92,6 @@
   <inertial>
       <origin xyz="0 0 0" rpy="0 0 0" />
-      <mass value="1" />
-      <xacro:cylinder_inertia mass="1" r="0.05" l="0.1" />
+      <mass value="0.1" />
+      <xacro:cylinder_inertia m="0.1" r="0.05" h="0.1" />
   </inertial>
   <visual>
@@ -140,7 +140,67 @@
   </collision>
  </link>
-  <xacro:link_wheel name="link_right_wheel" />
-  <xacro:joint_wheel name="joint_right_wheel" child="link_right_wheel" origin_xyz="-0.05 0.15 0" />
-  <xacro:link_wheel name="link_left_wheel" />
-  <xacro:joint_wheel name="joint_left_wheel" child="link_left_wheel" origin_xyz="-0.05 -0.15 0" />
+ <link name="left_wheel">
+   <!--origin xyz="0.1 0.13 0.1" rpy="0 1.5707 1.5707"/-->
+   <collision name="collision">
+     <origin xyz="0 0 0" rpy="0 1.5707 1.5707"/>
+     <geometry>
+       <cylinder radius="0.1" length="0.05"/>
+     </geometry>
+   </collision>
+   <visual name="left_wheel_visual">
+     <origin xyz="0 0 0" rpy="0 1.5707 1.5707"/>
+     <geometry>
+       <cylinder radius="0.1" length="0.05"/>
+     </geometry>
+   </visual>
+   <inertial>
+     <origin xyz="0 0 0" rpy="0 1.5707 1.5707"/>
+     <mass value="5"/>
+     <cylinder_inertia m="5" r="0.1" h="0.05"/>
+     <inertia
+       ixx="1.0" ixy="0.0" ixz="0.0"
+       iyy="1.0" iyz="0.0"
+       izz="1.0"/>
+   </inertial>
+ </link>
+ <link name="right_wheel">
+   <!--origin xyz="0.1 -0.13 0.1" rpy="0 1.5707 1.5707"/-->
+   <collision name="collision">
+     <origin xyz="0 0 0" rpy="0 1.5707 1.5707"/>
+     <geometry>
+       <cylinder radius="0.1" length="0.05"/>
+     </geometry>
+   </collision>
+   <visual name="right_wheel_visual">
+     <origin xyz="0 0 0" rpy="0 1.5707 1.5707"/>
+     <geometry>
+       <cylinder radius="0.1" length="0.05"/>
+     </geometry>
+   </visual>
+   <inertial>
+     <origin xyz="0 0 0" rpy="0 1.5707 1.5707"/>
+     <mass value="5"/>
+     <cylinder_inertia m="5" r="0.1" h="0.05"/>
+     <inertia
+       ixx="1.0" ixy="0.0" ixz="0.0"
+       iyy="1.0" iyz="0.0"
+       izz="1.0"/>
+   </inertial>
+ </link>
+ <joint type="continuous" name="left_wheel_hinge">
+   <origin xyz="-0.1 0.15 0" rpy="0 0 0"/>
+   <child link="left_wheel"/>
+   <parent link="link_chassis"/>
+   <axis xyz="0 1 0" rpy="0 0 0"/>
+   <limit effort="100" velocity="100"/>
+   <joint_properties damping="0.0" friction="0.0"/>
+ </joint>
+ <joint type="continuous" name="right_wheel_hinge">
+   <origin xyz="-0.1 -0.15 0" rpy="0 0 0"/>
+   <child link="right_wheel"/>
+   <parent link="link_chassis"/>
+   <axis xyz="0 1 0" rpy="0 0 0"/>
+   <limit effort="100" velocity="100"/>
+   <joint_properties damping="0.0" friction="0.0"/>
+ </joint>
 </robot>
